File: Circuit/TempViewer V1.0/Analogverarbeitung.kicad_sch (KiCad schematic)
At the start: 39 parts, among them U1 LTC2451xDDB, U10 ATA00AA36S-L, U11 TLV1117-33, U13 LTC1798CS8-3PBF, U4 MAX4289ESA+, U5 MAX4289ESA+, U6 ISO1641BDR, U7 AD5272BCP, U8 AD5272BCP, U9 TLP2770

Commit message: Update
Parts:
- added C20, C21, C22, C23: C, symbol Device:C
- added J1: Screw_Terminal_01x02, TerminalBlock_TE-Connectivity:TerminalBlock_TE_282834-2_1x02_P2.54mm_Horizontal, symbol Connector:Screw_Terminal_01x02
- added JP7, JP8: SolderJumper_2_Open, Jumper:SolderJumper-2_P1.3mm_Open_RoundedPad1.0x1.5mm, symbol Jumper:SolderJumper_2_Open
- added U12: LTC1798CS8-3PBF, symbol TempViewerLIB:LTC1798CS8-3PBF
Connections:
- net -VREF: now also C22.2, C23.1, JP7.2 (B); no longer C18.2, C19.1, U1.2 (REF-), U7.2 (A), U8.2 (A)
- net A-5V: now also U12.4 (GND)
- net AGND: now also C20.2, C21.2, J1.2 (Pin_2), U12.2 (IN)
- net GND: now also JP8.1 (A)
- net Thermoelement+: now also J1.1 (Pin_1)
- net at U7.5 (EXT_CAP): now also C20.1
- net at U8.5 (EXT_CAP): now also C21.1
- new net AR1.1: C18.2, C19.1, C22.1, C23.2, JP7.1 (A), JP8.2 (B), U1.2 (REF-), U12.6 (OUT), U7.2 (A), U8.2 (A)
Other:
- note added: "3V AnalogDigital"
- note added: "AnalogReferenz"

Commit message: Update
Parts:
- removed C22, C23: C, symbol Device:C
- removed U12: LTC1798CS8-3PBF, symbol TempViewerLIB:LTC1798CS8-3PBF
- added JP10, JP9: SolderJumper_2_Open, Jumper:SolderJumper-2_P1.3mm_Open_RoundedPad1.0x1.5mm, symbol Jumper:SolderJumper_2_Open
- added R27, R28: R, Resistor_SMD:R_0603_1608Metric, symbol Device:R
- C10, C11, C14, C15, C16, C17, C18, C7, C8, C9: value C -> 100nF; footprint (none) -> Capacitor_SMD:C_0805_2012Metric
- C12, C13: value C_Polarized -> 470uF; footprint (none) -> Capacitor_SMD:CP_Elec_8x6.7
- C19: value C -> 10nF; footprint (none) -> Capacitor_SMD:C_0805_2012Metric
- C20, C21, C5, C6: footprint (none) -> Capacitor_SMD:C_0805_2012Metric
- R10, R9: footprint (none) -> Resistor_SMD:R_0805_2012Metric
- U11: footprint (none) -> Package_TO_SOT_SMD:SOT-223
- U13, U6: footprint (none) -> Package_SO:SOIC-8_3.9x4.9mm_P1.27mm
- U4, U5: value MAX4289ESA+ -> MAX4289ESA+ / OP37; footprint (none) -> Package_SO:SOIC-8_3.9x4.9mm_P1.27mm
Connections:
- net -VREF: no longer U5.4 (GND)
- net A3V3: now also U4.7 (VCC), U5.4 (GND)
- net AGND: now also JP8.1 (A)
- net AR2.1: now also JP10.1 (A), R28.1
- net GND: no longer JP8.1 (A)
- net VREF: no longer U4.7 (VCC)
- net at C6.1, R10.2, U1.6 (IN): now also JP10.2 (B), R28.2
- net at D3.2 (A), D4.1 (K), R9.1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: now also JP9.1 (A), R27.1
- net at C5.1, R9.2, U5.3 (IN+): now also JP9.2 (B), R27.2
