File: Circuit/TempViewer V1.0/MCU.kicad_sch (KiCad schematic)
At the start: 20 parts, among them Q1 DMN3731U, Q2 DMN3731U, U2 PIC16F18877-I/PT

Commit message: Analog Circuits added
Parts:
- Q1, Q2: footprint MySmd:TRANS_BC847B -> Package_TO_SOT_SMD:SOT-23
- R1, R3: value 180R -> 1KR
Connections:
- net Interlock_2: no longer U2.43 (RC5), U2.44 (RC6)
- new net Interlock_3: U2.43 (RC5)
- new net Interlock_4: U2.44 (RC6)
Changed lines of the file:
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@@
     )
   )
-  (global_label "Interlock_2" (shape input) (at 115.57 29.21 0) (fields_autoplaced)
+  (global_label "Interlock_4" (shape input) (at 115.57 29.21 0) (fields_autoplaced)
     (effects (font (size 1.27 1.27)) (justify left))
     (property "Intersheetrefs" "${INTERSHEET_REFS}" (at 129.0175 29.21 0)
@@
     )
   )
-  (global_label "Interlock_2" (shape input) (at 115.57 31.75 0) (fields_autoplaced)
+  (global_label "Interlock_3" (shape input) (at 115.57 31.75 0) (fields_autoplaced)
     (effects (font (size 1.27 1.27)) (justify left))
     (property "Intersheetrefs" "${INTERSHEET_REFS}" (at 129.0175 31.75 0)
@@
       (effects (font (size 1.27 1.27)) (justify left))
     )
-    (property "Footprint" "MySmd:TRANS_BC847B" (at 29.21 136.525 0)
+    (property "Footprint" "Package_TO_SOT_SMD:SOT-23" (at 29.21 136.525 0)
       (effects (font (size 1.27 1.27) italic) (justify left) hide)
     )
-    (property "Datasheet" "https://www.diodes.com/assets/Datasheets/DMN3731U.pdf" (at 24.13 134.62 0)
+    (property "Datasheet" "http://www.diodes.com/assets/Datasheets/ds31181.pdf" (at 24.13 134.62 0)
       (effects (font (size 1.27 1.27)) (justify left) hide)
     )
@@
       (effects (font (size 1.27 1.27)) (justify right))
     )
-    (property "Value" "180R" (at 46.99 127 0)
+    (property "Value" "1KR" (at 46.99 127 0)
       (effects (font (size 1.27 1.27)) (justify right))
     )
@@
       (effects (font (size 1.27 1.27)) (justify left))
     )
-    (property "Footprint" "MySmd:TRANS_BC847B" (at 57.15 136.525 0)
+    (property "Footprint" "Package_TO_SOT_SMD:SOT-23" (at 57.15 136.525 0)
       (effects (font (size 1.27 1.27) italic) (justify left) hide)
     )
-    (property "Datasheet" "https://www.diodes.com/assets/Datasheets/DMN3731U.pdf" (at 52.07 134.62 0)
+    (property "Datasheet" "http://www.diodes.com/assets/Datasheets/ds31181.pdf" (at 52.07 134.62 0)
       (effects (font (size 1.27 1.27)) (justify left) hide)
     )
@@
       (effects (font (size 1.27 1.27)) (justify right))
     )
-    (property "Value" "180R" (at 19.05 127 0)
-      (effects (font (size 1.27 1.27)) (justify right))
-    )
+    (property "Value" "1KR" (at 19.05 127 0)
+      (effects (font (size 1.27 1.27)) (justify right))
+    )

Commit message: Update
Parts:
- added J3: Programming, Connector_PinHeader_2.54mm:PinHeader_1x06_P2.54mm_Vertical, symbol Connector:Conn_01x06_Pin
- S1: footprint MySmd:SW_DS04-254-2-04BK-SMT-TR -> MY_SMD_LIB:SW_DS04-254-2-04BK-SMT-TR
- U2: footprint MySmd:TQFP44_PT_MCH -> Package_QFP:TQFP-44_10x10mm_P0.8mm
- U3: footprint MySmd:RH100 -> MY_SMD_LIB:XTAL_ABM8-37.500MHZ-12-1-U-T
Connections:
- net 5V: now also J3.5 (Pin_5)
- net GND: now also J3.4 (Pin_4)
- net at U2.16 (RB6/ICSPCLK): now also J3.2 (Pin_2)
- net at U2.17 (RB7/ICSPDAT): now also J3.3 (Pin_3)
- net at U2.18 (RE3/*MCLR/VPP): now also J3.6 (Pin_6)
Changed lines of the file:
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@@
+    (stroke (width 0) (type default))
+  )
+  (wire (pts (xy 27.94 69.85) (xy 34.29 69.85))
     (stroke (width 0) (type default))
   )
@@
     (stroke (width 0) (type default))
   )
+  (wire (pts (xy 27.94 67.31) (xy 34.29 67.31))
+    (stroke (width 0) (type default))
+  )
   (wire (pts (xy 83.82 143.51) (xy 83.82 146.05))
     (stroke (width 0) (type default))
@@
     (stroke (width 0) (type default))
   )
+  (wire (pts (xy 55.88 69.85) (xy 43.18 69.85))
+    (stroke (width 0) (type default))
+  )
   (wire (pts (xy 19.05 186.69) (xy 19.05 182.88))
     (stroke (width 0) (type default))
@@
     (stroke (width 0) (type default))
   )
+  (wire (pts (xy 27.94 62.23) (xy 45.72 62.23))
+    (stroke (width 0) (type default))
+  )
   (wire (pts (xy 138.43 60.96) (xy 138.43 62.23))
     (stroke (width 0) (type default))
@@
     (stroke (width 0) (type default))
   )
+  (wire (pts (xy 43.18 64.77) (xy 27.94 64.77))
+    (stroke (width 0) (type default))
+  )
   (wire (pts (xy 223.52 109.22) (xy 223.52 111.76))
     (stroke (width 0) (type default))
@@
     (stroke (width 0) (type default))
   )
+  (wire (pts (xy 45.72 67.31) (xy 55.88 67.31))
+    (stroke (width 0) (type default))
+  )
   (wire (pts (xy 115.57 143.51) (xy 115.57 160.02))
     (stroke (width 0) (type default))
@@
     (stroke (width 0) (type default))
   )
+  (wire (pts (xy 45.72 62.23) (xy 45.72 67.31))
+    (stroke (width 0) (type default))
+  )
   (wire (pts (xy 49.53 49.53) (xy 55.88 49.53))
     (stroke (width 0) (type default))
@@
     (stroke (width 0) (type default))
   )
+  (wire (pts (xy 43.18 69.85) (xy 43.18 64.77))
+    (stroke (width 0) (type default))
+  )
   (wire (pts (xy 107.95 143.51) (xy 115.57 143.51))
     (stroke (width 0) (type default))
@@
     (stroke (width 0) (type default))
   )
+  (wire (pts (xy 27.94 72.39) (xy 55.88 72.39))
+    (stroke (width 0) (type default))
+  )
   (wire (pts (xy 55.88 82.55) (xy 50.8 82.55))
     (stroke (width 0) (type default))
@@
     )
   )
+  (global_label "GND" (shape input) (at 34.29 67.31 0) (fields_autoplaced)
+    (effects (font (size 1.27 1.27)) (justify left))
+    (property "Intersheetrefs" "${INTERSHEET_REFS}" (at 41.1457 67.31 0)
+      (effects (font (size 1.27 1.27)) (justify left) hide)
+    )
+  )
   (global_label "ADDR_3" (shape input) (at 203.2 81.28 180) (fields_autoplaced)
     (effects (font (size 1.27 1.27)) (justify right))
@@
     (property "Intersheetrefs" "${INTERSHEET_REFS}" (at 26.67 152.9057 90)
       (effects (font (size 1.27 1.27)) (justify right) hide)
+    )
+  )
+  (global_label "5V" (shape input) (at 34.29 69.85 0) (fields_autoplaced)
+    (effects (font (size 1.27 1.27)) (justify left))
+    (property "Intersheetrefs" "${INTERSHEET_REFS}" (at 39.5733 69.85 0)
+      (effects (font (size 1.27 1.27)) (justify left) hide)
     )
   )
@@
     )
   )
+  (symbol (lib_id "Connector:Conn_01x06_Pin") (at 22.86 64.77 0) (unit 1)
+    (in_bom yes) (on_board yes) (dnp no) (fields_autoplaced)
+    (property "Reference" "J3" (at 23.495 54.61 0)
+      (effects (font (size 1.27 1.27)))
+    )
+    (property "Value" "Programming" (at 23.495 57.15 0)
+      (effects (font (size 1.27 1.27)))
+    )
+    (property "Footprint" "Connector_PinHeader_2.54mm:PinHeader_1x06_P2.54mm_Vertical" (at 22.86 64.77 0)
+      (effects (font (size 1.27 1.27)) hide)
+    )
+    (property "Datasheet" "~" (at 22.86 64.77 0)
+      (effects (font (size 1.27 1.27)) hide)
+    )
+    (pin "2")
+    (pin "1")
+    (pin "5")
+    (pin "3")
+    (pin "6")
+    (pin "4")
+    (instances
+      (project "TempViewer V1.0"
+        (path "/9be733a6-d9bf-4549-8c43-ef6367cdf2b9/6d9aa1b9-eca4-43e5-baa7-e762d6b2948a"
+          (reference "J3") (unit 1)
+        )
+      )
+    )
+  )
   (symbol (lib_id "MYLIB_2:DS04-254-2-04BK-SMT-TR") (at 100.33 143.51 0) (unit 1)
     (in_bom yes) (on_board yes) (dnp no) (fields_autoplaced)
@@
       (effects (font (size 1.27 1.27)))
     )
-    (property "Footprint" "MySmd:SW_DS04-254-2-04BK-SMT-TR" (at 100.33 143.51 0)
+    (property "Footprint" "MY_SMD_LIB:SW_DS04-254-2-04BK-SMT-TR" (at 100.33 143.51 0)
       (effects (font (size 1.27 1.27)) (justify bottom) hide)
     )
@@
       (effects (font (size 1.27 1.27)))
     )
-    (property "Footprint" "MySmd:RH100" (at 26.67 172.72 0)
+    (property "Footprint" "MY_SMD_LIB:XTAL_ABM8-37.500MHZ-12-1-U-T" (at 26.67 172.72 0)
       (effects (font (size 1.27 1.27)) hide)
     )
@@
       (effects (font (size 1.524 1.524)))
     )
-    (property "Footprint" "MySmd:TQFP44_PT_MCH" (at 55.88 29.21 0)
+    (property "Footprint" "Package_QFP:TQFP-44_10x10mm_P0.8mm" (at 55.88 29.21 0)
       (effects (font (size 1.27 1.27) italic) hide)
     )
