File: Circuit/TempViewer V1.0/DigitalPower.kicad_sch (KiCad schematic)
At the start: 0 parts

Commit message: Update
Parts:
- added C24: 470uF, Capacitor_SMD:CP_Elec_10x10, symbol Device:C_Polarized
- added C25: 470uF, Capacitor_SMD:CP_Elec_8x6.7, symbol Device:C_Polarized
- added C26, C27, C28, C29: 100nF, Capacitor_SMD:C_0805_2012Metric, symbol Device:C
- added D15, D16: LED, LED_SMD:LED_1206_3216Metric, symbol Device:LED
- added J2: 12V IN, TerminalBlock_Phoenix:TerminalBlock_Phoenix_MKDS-3-2-5.08_1x02_P5.08mm_Horizontal, symbol Connector:Screw_Terminal_01x02
- added J4: 12V OUT, TerminalBlock_Phoenix:TerminalBlock_Phoenix_MKDS-3-2-5.08_1x02_P5.08mm_Horizontal, symbol Connector:Screw_Terminal_01x02
- added J5: 5V IN, TerminalBlock_Phoenix:TerminalBlock_Phoenix_MKDS-3-2-5.08_1x02_P5.08mm_Horizontal, symbol Connector:Screw_Terminal_01x02
- added J6: I2C, TerminalBlock_Phoenix:TerminalBlock_Phoenix_MKDS-3-2-5.08_1x02_P5.08mm_Horizontal, symbol Connector:Screw_Terminal_01x02
- added J7: 5V OUT, TerminalBlock_Phoenix:TerminalBlock_Phoenix_MKDS-3-2-5.08_1x02_P5.08mm_Horizontal, symbol Connector:Screw_Terminal_01x02
- added R25: R, Resistor_SMD:R_1206_3216Metric, symbol Device:R
- added R26: 180R, Resistor_SMD:R_1206_3216Metric, symbol Device:R
- added U14: LM7805_TO220, Package_TO_SOT_THT:TO-220-3_Vertical, symbol Regulator_Linear:LM7805_TO220
Connections:
- new net: D16.2 (A), R26.2
- new net: D15.2 (A), R25.2
- new net 12V: C24.1, C28.1, C29.2, J2.1 (Pin_1), J4.1 (Pin_1), R25.1, U14.1 (VI)
- new net 5V: C25.1, C26.1, C27.2, J5.1 (Pin_1), J7.1 (Pin_1), R26.1, U14.3 (VO)
- new net GND: C24.2, C25.2, C26.2, C27.1, C28.2, C29.1, D15.1 (K), D16.1 (K), J2.2 (Pin_2), J4.2 (Pin_2), J5.2 (Pin_2), J7.2 (Pin_2), U14.2 (GND)
- new net SCL: J6.1 (Pin_1)
- new net SDA: J6.2 (Pin_2)

Commit message: PCB Design V1
Parts:
- added J12: PE, TerminalBlock_Phoenix:TerminalBlock_Phoenix_MKDS-3-2-5.08_1x02_P5.08mm_Horizontal, symbol Connector:Screw_Terminal_01x02
Connections:
- new net PE: J12.1 (Pin_1), J12.2 (Pin_2)
Changed lines of the file:
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@@
   (junction (at 40.64 58.42) (diameter 0) (color 0 0 0 0)
   )
+  (junction (at 54.61 20.32) (diameter 0) (color 0 0 0 0)
+  )
   (junction (at 50.8 73.66) (diameter 0) (color 0 0 0 0)
   )
@@
     (stroke (width 0) (type default))
   )
+  (wire (pts (xy 54.61 22.86) (xy 54.61 20.32))
+    (stroke (width 0) (type default))
+  )
   (wire (pts (xy 50.8 71.12) (xy 50.8 73.66))
     (stroke (width 0) (type default))
@@
     (stroke (width 0) (type default))
   )
+  (wire (pts (xy 55.88 22.86) (xy 54.61 22.86))
+    (stroke (width 0) (type default))
+  )
   (wire (pts (xy 57.15 40.64) (xy 67.31 40.64))
     (stroke (width 0) (type default))
@@
     (stroke (width 0) (type default))
   )
+  (wire (pts (xy 54.61 20.32) (xy 55.88 20.32))
+    (stroke (width 0) (type default))
+  )
   (wire (pts (xy 58.42 71.12) (xy 58.42 73.66))
     (stroke (width 0) (type default))
@@
   )
   (wire (pts (xy 50.8 111.76) (xy 60.96 111.76))
+    (stroke (width 0) (type default))
+  )
+  (wire (pts (xy 53.34 20.32) (xy 54.61 20.32))
     (stroke (width 0) (type default))
   )
@@
     )
   )
+  (global_label "PE" (shape input) (at 53.34 20.32 180) (fields_autoplaced)
+    (effects (font (size 1.27 1.27)) (justify right))
+    (property "Intersheetrefs" "${INTERSHEET_REFS}" (at 47.9358 20.32 0)
+      (effects (font (size 1.27 1.27)) (justify right) hide)
+    )
+  )
   (global_label "GND" (shape input) (at 133.35 46.99 0) (fields_autoplaced)
     (effects (font (size 1.27 1.27)) (justify left))
@@
         )
       )
+    )
+  )
+  (symbol (lib_id "Connector:Screw_Terminal_01x02") (at 60.96 20.32 0) (unit 1)
+    (in_bom yes) (on_board yes) (dnp no) (fields_autoplaced)
+    (property "Reference" "J12" (at 60.96 29.21 0)
+      (effects (font (size 1.27 1.27)) hide)
+    )
+    (property "Value" "PE" (at 63.5 21.59 0)
+      (effects (font (size 1.27 1.27)) (justify left))
+    )
+    (property "Footprint" "TerminalBlock_Phoenix:TerminalBlock_Phoenix_MKDS-3-2-5.08_1x02_P5.08mm_Horizontal" (at 60.96 20.32 0)
+      (effects (font (size 1.27 1.27)) hide)
+    )
+    (property "Datasheet" "~" (at 60.96 20.32 0)
+      (effects (font (size 1.27 1.27)) hide)
+    )
+    (pin "2")
+    (pin "1")
+    (instances
+      (project "TempViewer V1.0"
+        (path "/9be733a6-d9bf-4549-8c43-ef6367cdf2b9/a2cad988-5f06-42bc-b673-20d9a8512d32"
+          (reference "J12") (unit 1)
+        )
+      )
